Commit message: check_wheel_control_train_fourth

File: data/Robots/Unitree/Go2W-Piper/go2w_piper_description/urdf/go2w_piper_description.urdf (robot description, URDF)
Before this commit: robot go2w_piper_description, 39 links, 38 joints
Links:
- added link Head_lower, mass 0.001; collision sphere radius=0.06
- added link Head_upper, mass 0.001; collision sphere radius=0.06
- added link imu, mass 0
- added link radar, mass 0
- link FL_calf: geometry collision box size=0.026 0.026 0.12; visual mesh filename=package://go2w_description/meshes/calf.stl
- link FL_calflower: geometry collision box size=0.022 0.022 0.065
- link FL_calflower1: geometry collision box size=0.031 0.031 0.03
- link FL_foot: geometry collision cylinder length=0.045 radius=0.086; visual mesh filename=package://go2w_description/meshes/left_wheel.dae
- link FL_foot_motor: geometry 
- link FL_hip: geometry collision sphere radius=0.046; visual mesh filename=package://go2w_description/meshes/hip.dae
- link FL_thigh: geometry collision box size=0.11 0.0245 0.034; visual mesh filename=package://go2w_description/meshes/thigh.dae
- link FR_calf: geometry collision box size=0.026 0.026 0.12; visual mesh filename=package://go2w_description/meshes/calf_mirror.stl
- link FR_calflower: geometry collision box size=0.022 0.022 0.065
- link FR_calflower1: geometry collision box size=0.031 0.031 0.03
- link FR_foot: geometry collision cylinder length=0.045 radius=0.086; visual mesh filename=package://go2w_description/meshes/right_wheel.dae
- link FR_foot_motor: geometry 
- link FR_hip: geometry collision sphere radius=0.046; visual mesh filename=package://go2w_description/meshes/hip.dae
- link FR_thigh: geometry collision box size=0.11 0.0245 0.034; visual mesh filename=package://go2w_description/meshes/thigh_mirror.dae
- link RL_calf: geometry collision box size=0.026 0.026 0.12; visual mesh filename=package://go2w_description/meshes/calf.stl
- link RL_calflower: geometry collision box size=0.022 0.022 0.065
- link RL_calflower1: geometry collision box size=0.031 0.031 0.03
- link RL_foot: geometry collision cylinder length=0.045 radius=0.086; visual mesh filename=package://go2w_description/meshes/left_wheel.dae
- link RL_foot_motor: geometry 
- link RL_hip: geometry collision sphere radius=0.046; visual mesh filename=package://go2w_description/meshes/hip.dae
- link RL_thigh: geometry collision box size=0.11 0.0245 0.034; visual mesh filename=package://go2w_description/meshes/thigh.dae
- link RR_calf: geometry collision box size=0.026 0.026 0.12; visual mesh filename=package://go2w_description/meshes/calf_mirror.stl
- link RR_calflower: geometry collision box size=0.022 0.022 0.065
- link RR_calflower1: geometry collision box size=0.031 0.031 0.03
- link RR_foot: geometry collision cylinder length=0.045 radius=0.086; visual mesh filename=package://go2w_description/meshes/right_wheel.dae
- link RR_foot_motor: geometry 
- link RR_hip: geometry collision sphere radius=0.046; visual mesh filename=package://go2w_description/meshes/hip.dae
- link RR_thigh: geometry collision box size=0.11 0.0245 0.034; visual mesh filename=package://go2w_description/meshes/thigh_mirror.dae
- link base: geometry collision box size=0.3762 0.0935 0.114; visual mesh filename=package://go2w_description/meshes/base.dae
Joints:
- added joint Head_lower_joint: type fixed, parent Head_upper, child Head_lower, origin xyz=0.008 0 -0.07 rpy=0 0 0, axis 0 0 0
- added joint Head_upper_joint: type fixed, parent base, child Head_upper, origin xyz=0.285 0 0.01 rpy=0 0 0, axis 0 0 0
- added joint imu_joint: type fixed, parent base, child imu, origin xyz=-0.02557 0 0.04232 rpy=0 0 0, axis 0 0 0
- added joint radar_joint: type fixed, parent base, child radar, origin xyz=0.28945 0 -0.046825 rpy=0 2.8782 0, axis 0 0 0
- joint FL_foot_joint: type revolute -> continuous
- joint FR_foot_joint: type revolute -> continuous
- joint RL_foot_joint: type revolute -> continuous
- joint RR_foot_joint: type revolute -> continuous
